Commit message: edit xacro to show link4.
launch gz create node brigde, pose, joint, ...

File: assign1/urdf/scara.urdf (robot description, URDF)
Before this commit: robot scara_robot, 6 links, 5 joints
Links:
- removed link link4
- link base_link: mass 10 -> None; geometry 
- link link1: mass 0.01 -> 10
- link link3: geometry collision box size=0.2 0.2 0.5; collision cylinder length=0.19999999999999998 radius=0.05
Joints:
- removed joint joint4
- joint joint1: origin xyz=0 0 0.1 rpy=0 0 0 -> xyz=0 0 0 rpy=0 0 0

File: assign1/urdf/scara.urdf copy.xacro (robot description, xacro)
@@ -1,16 +1,4 @@
 <?xml version="1.0"?>
 <robot name="scara_robot" xmlns:xacro="http://www.ros.org/wiki/xacro">
-    <material name="blue">
-        <color rgba="0 0 0.8 1"/>
-    </material>
-    <material name="red">
-        <color rgba="0.8 0 0 1"/>
-    </material>
-    <material name="green">
-        <color rgba="0.0 1.0 0.0 1.0"/>
-    </material>
-    <material name="purple">
-        <color rgba="0.5 0.0 0.5 1.0"/>
-    </material>
     <xacro:property name="d1" value=".6" />
     <xacro:property name="a1" value=".6" />
@@ -30,10 +18,9 @@
     <xacro:property name="link1_r" value="${link_r}" />
     <xacro:property name="link1_theta" value="0" />
-    <!-- <xacro:property name="link1_d" value="${base_link_h}" /> -->
-     <xacro:property name="link1_d" value="0" />
+    <xacro:property name="link1_d" value="${base_link_h}" />
     <xacro:property name="link1_a" value="0" />
     <xacro:property name="link1_alpha" value="0" />
     <xacro:property name="link1_arm_l" value="${a1}" />
-    <xacro:property name="link1_arm_w" value="${link_r}" />
+    <xacro:property name="link1_arm_w" value="${link_r *2}" />
     <xacro:property name="link1_arm_h" value="${link_r}" />
     <xacro:property name="link2_l" value="${cyl_joint_l}" />
@@ -44,5 +31,5 @@
     <xacro:property name="link2_alpha" value="0" />
     <xacro:property name="link2_arm_l" value="${a2}" />
-    <xacro:property name="link2_arm_w" value="${link_r}" />
+    <xacro:property name="link2_arm_w" value="${link_r *2}" />
     <xacro:property name="link2_arm_h" value="${link_r}" />
     <xacro:property name="link3_arm_l" value="${prismatic_link_a}" />
@@ -98,5 +85,5 @@
             </geometry>
         </collision>
-        <xacro:inertial_box mass="100" x="${base_link_l}" y="${base_link_w}" z="${base_link_h}">
+        <xacro:inertial_box mass="10" x="${base_link_l}" y="${base_link_w}" z="${base_link_h}">
             <origin rpy="0 0 0" xyz="0 0 ${base_link_h/2}" />
         </xacro:inertial_box>
@@ -108,5 +95,5 @@
         <axis xyz="0 0 1" />
         <limit lower="${-5*pi/6}" upper="${5*pi/6}" effort="100" velocity="5.0" />
-        <dynamics damping="0.1" friction="0.0"/>
+        <dynamics damping="0.1" friction="0.1"/>
     </joint>
     <link name="link1">
@@ -116,13 +103,12 @@
                 <cylinder length="${link1_l}" radius="${link1_r}" />
             </geometry>
-            <material name="green"/>
-        </visual>
-        <collision>
-            <origin rpy="0 0 0" xyz="0 0 ${link1_l/2 + base_link_h/2}" />
-            <geometry>
-                <cylinder length="${link1_l - base_link_h}" radius="${link1_r}" />
-            </geometry>
-        </collision>
-        <xacro:inertial_cylinder mass="1" length="${link1_l}" radius="${link1_r}">
+        </visual>
+        <collision>
+            <origin rpy="0 0 0" xyz="0 0 ${link1_l/2}" />
+            <geometry>
+                <cylinder length="${link1_l}" radius="${link1_r}" />
+            </geometry>
+        </collision>
+        <xacro:inertial_cylinder mass="10" length="${link1_l}" radius="${link1_r}">
             <origin rpy="0 0 0" xyz="0 0 ${link1_l/2}" />
         </xacro:inertial_cylinder>
@@ -139,5 +125,5 @@
             </geometry>
         </collision>
-        <xacro:inertial_box mass="0.5" x="${link1_arm_l}" y="${link1_arm_w}" z="${link1_arm_h}">
+        <xacro:inertial_box mass="0.01" x="${link1_arm_l}" y="${link1_arm_w}" z="${link1_arm_h}">
             <origin rpy="0 0 0" xyz="${link1_arm_l/2} 0 0" />
         </xacro:inertial_box>
@@ -149,5 +135,4 @@
                 <cylinder length="${link2_l}" radius="${link2_r}" />
             </geometry>
-            <material name="blue"/>
         </visual>
         <collision>
@@ -157,5 +142,5 @@
             </geometry>
         </collision>
-        <xacro:inertial_cylinder mass="0.5" length="${link2_l}" radius="${link2_r}">
+        <xacro:inertial_cylinder mass="0.01" length="${link2_l}" radius="${link2_r}">
             <origin rpy="0 0 0" xyz="0 0 0" />
         </xacro:inertial_cylinder>
@@ -172,5 +157,5 @@
             </geometry>
         </collision>
-        <xacro:inertial_box mass="0.5" x="${link2_arm_l}" y="${link2_arm_w}" z="${link2_arm_h}">
+        <xacro:inertial_box mass="0.01" x="${link2_arm_l}" y="${link2_arm_w}" z="${link2_arm_h}">
             <origin rpy="0 0 0" xyz="${link2_arm_l/2} 0 0" />
         </xacro:inertial_box>
@@ -189,5 +174,4 @@
                 <box size="${link3_arm_l} ${link3_arm_w} ${link3_arm_h}" />
             </geometry>
-            <material name="red"/>
         </visual>
         <collision>
@@ -197,7 +181,22 @@
             </geometry>
         </collision>
-        <xacro:inertial_box mass="0.5" x="${link3_arm_l}" y="${link3_arm_w}" z="${link3_arm_h}">
+        <xacro:inertial_box mass="0.01" x="${link3_arm_l}" y="${link3_arm_w}" z="${link3_arm_h}">
             <origin rpy="0 0 0" xyz="0 0 ${link3_arm_h/2 - prismatic_link_a/2}" />
         </xacro:inertial_box>
+        <visual>
+            <origin rpy="0 0 0" xyz="0 0 ${-link4_l/2}" />
+            <geometry>
+                <cylinder length="${link4_l}" radius="${link4_r}" />
+            </geometry>
+        </visual>
+        <collision>
+            <origin rpy="0 0 0" xyz="0 0 ${-(link4_l - prismatic_link_a/2)/2}" />
+            <geometry>
+                <cylinder length="${link4_l - prismatic_link_a/2}" radius="${link4_r}" />
+            </geometry>
+        </collision>
+        <xacro:inertial_cylinder mass="0.01" length="${link4_l}" radius="${link4_r}">
+            <origin rpy="0 0 0" xyz="0 0 ${-link4_l/2}" />
+        </xacro:inertial_cylinder>
     </link>
     <joint name="joint3" type="prismatic">
@@ -208,5 +207,5 @@
         <axis xyz="0 0 -1" />
     </joint>
-    <link name="link4">
+    <!-- <link name="link4">
         <visual>
             <origin rpy="0 0 0" xyz="0 0 ${-link4_l/2}" />
@@ -214,5 +213,4 @@
                 <cylinder length="${link4_l}" radius="${link4_r}" />
             </geometry>
-            <material name="purple"/>
         </visual>
         <collision>
@@ -222,16 +220,16 @@
             </geometry>
         </collision>
-        <xacro:inertial_cylinder mass="0.5" length="${link4_l}" radius="${link4_r}">
+        <xacro:inertial_cylinder mass="0.01" length="${link4_l}" radius="${link4_r}">
             <origin rpy="0 0 0" xyz="0 0 ${-link4_l/2}" />
         </xacro:inertial_cylinder>
     </link>
-    <joint name="joint4" type="fixed">
+    <joint name="joint4" type="continuous">
         <parent link="link3" />
         <child link="link4" />
         <origin rpy="${link4_alpha} 0 ${link4_theta}" xyz="0 0 ${link4_d}" />
         <axis xyz="0 0 1" />
-    </joint>
+    </joint> -->
      <!-- Use for GUI control -->
-    <gazebo>
+    <!-- <gazebo>
         <plugin filename="gz-sim-joint-position-controller-system"
             name="gz::sim::systems::JointPositionController">
@@ -252,9 +250,5 @@
             <cmd_max>1.0</cmd_max>
         </plugin>
-    </gazebo>
-    <!-- Set joint4 to publish, it is fixed joint which will not publish by default-->
-    <gazebo reference="joint4">
-        <preserveFixedJoint>true</preserveFixedJoint>
-    </gazebo>
+    </gazebo> -->
     <gazebo>
         <plugin
@@ -274,5 +268,5 @@
             <use_pose_vector_msg>true</use_pose_vector_msg>
         </plugin>
-        <!-- <plugin
+        <plugin
             filename="ignition-gazebo-joint-trajectory-controller-system"
             name="ignition::gazebo::systems::JointTrajectoryController">
@@ -305,5 +299,5 @@
             <position_cmd_max>50</position_cmd_max>
             <position_cmd_max>50</position_cmd_max>
-        </plugin> -->
+        </plugin>
     </gazebo>
 </robot>
