Commit message: added plugin manager for model

File: src/assign2/urdf/scara_fixed_joints_classic.urdf.xacro (robot description, xacro)
@@ -1,4 +1,5 @@
 <?xml version="1.0"?>
 <robot name="scara_robot" xmlns:xacro="http://www.ros.org/wiki/xacro">
+    <xacro:arg name="controllers_file" default="" />
     <!-- Joint colors-->
     <gazebo reference="link1">
@@ -11,7 +12,7 @@
         <material>Gazebo/Red</material>
     </gazebo>
-    <gazebo reference="link4">
+    <!-- <gazebo reference="link4">
         <material>Gazebo/Purple</material>
-    </gazebo>
+    </gazebo> -->
     <!-- Robot dimensions -->
     <xacro:property name="d1" value=".5" />
@@ -81,5 +82,5 @@
     <xacro:property name="link3_arm_w" value="${prismatic_link_a}" />
     <xacro:property name="link3_arm_h" value="${prismatic_link_a + prismatic_extend_range}" />
-    <xacro:property name="link3_arm_mass" value="2" />
+    <xacro:property name="link3_arm_mass" value="10" />
     <!-- DH data of joint 3-->
     <xacro:property name="link3_theta" value="0" />
@@ -143,11 +144,11 @@
         </xacro:inertial_box>
     </link>
-    <joint name="joint1" type="revolute">
+    <joint name="joint1" type="fixed">
         <parent link="base_link" />
         <child link="link1" />
         <origin rpy="0 0 0" xyz="0 0 ${link1_d}" />
         <axis xyz="0 0 1" />
-        <limit lower="${joint1_lower}" upper="${joint1_upper}" effort="100" velocity="5.0" />
-        <dynamics damping="0.5" friction="1"/>
+        <!-- <limit lower="${joint1_lower}" upper="${joint1_upper}" effort="100" velocity="5.0" />
+        <dynamics damping="0.5" friction="1"/> -->
     </joint>
     <link name="link1">
@@ -248,11 +249,11 @@
         <child link="link3" />
         <origin rpy="0 0 0" xyz="${link3_a} 0 0" />
-           <limit lower="${joint3_lower}" upper="${joint3_upper}" effort="100" velocity="5" />
+           <limit lower="${joint3_lower}" upper="${joint3_upper}" effort="1000" velocity="5" />
         <axis xyz="0 0 -1" />
-           <dynamics damping="5" friction="25"/>
+           <dynamics damping="10" friction="100"/>
     </joint>
-    <link name="link4">
+    <!-- <link name="link4"> -->
         <!-- Cylinder visual -->
-        <visual>
+        <!-- <visual>
             <origin rpy="0 0 0" xyz="0 0 ${-link4_l/2}" />
             <geometry>
@@ -275,18 +276,30 @@
         <origin rpy="${link4_alpha} 0 ${link4_theta}" xyz="0 0 ${link4_d}" />
         <axis xyz="0 0 1" />
-    </joint>
+    </joint> -->
     <!--
             Gazebo Classic configuration
      -->
+    <ros2_control name="GazeboSystem" type="system">
+        <hardware>
+            <plugin>gazebo_ros2_control/GazeboSystem</plugin>
+        </hardware>
+        <joint name="joint3">
+            <command_interface name="effort">
+                <param name="min">-1000</param>
+                <param name="max">1000</param>
+            </command_interface>
+            <state_interface name="position" />
+            <state_interface name="velocity" />
+            <state_interface name="effort" />
+        </joint>
+    </ros2_control>
     <!--
         /gazebo/apply_joint_effort is provided by gazebo_ros API when Gazebo Classic
-        is launched with gazebo_ros. This plugin publishes ROS joint states.
+        is launched with gazebo_ros. Joint states are published through ros2_control
+        and the joint_state_broadcaster config file instead of the old Gazebo plugin.
     -->
     <gazebo>
-        <plugin name="gazebo_ros_joint_state_publisher" filename="libgazebo_ros_joint_state_publisher.so">
-            <alwaysOn>true</alwaysOn>
-            <update_rate>50.0</update_rate>
-            <joint_name>joint1</joint_name>
-            <joint_name>joint3</joint_name>
+        <plugin name="gazebo_ros2_control" filename="libgazebo_ros2_control.so">
+            <parameters>$(arg controllers_file)</parameters>
         </plugin>
     </gazebo>
