Commit message: add ros_gz bridge for apply joint effort

File: src/assign2/urdf/scara_fixed_joints.urdf.xacro (robot description, xacro)
@@ -81,5 +81,5 @@
     <xacro:property name="link3_arm_w" value="${prismatic_link_a}" />
     <xacro:property name="link3_arm_h" value="${prismatic_link_a + prismatic_extend_range}" />
-    <xacro:property name="link3_arm_mass" value="2" />
+    <xacro:property name="link3_arm_mass" value="10" />
     <!-- DH data of joint 3-->
     <xacro:property name="link3_theta" value="0" />
@@ -90,5 +90,5 @@
     <xacro:property name="link4_l" value="${ee_l}" />
     <xacro:property name="link4_r" value="${ee_r}" />
-    <xacro:property name="link4_mass" value="0.5" />
+    <xacro:property name="link4_mass" value="1" />
     <!-- DH data of joint 4 -->
     <xacro:property name="link4_theta" value="0" />
@@ -251,11 +251,11 @@
         <child link="link3" />
         <origin rpy="0 0 0" xyz="${link3_a} 0 0" />
-        <limit lower="${joint3_lower}" upper="${joint3_upper}" effort="100" velocity="5" />
         <axis xyz="0 0 -1" />
-        <!-- <dynamics damping="0.5" friction="1"/> -->
+        <limit lower="${joint3_lower}" upper="${joint3_upper}" effort="1000" velocity="5" />
+        <dynamics damping="5" friction="100"/>
     </joint>
-    <link name="link4">
+    <!-- <link name="link4"> -->
         <!-- Cylinder visual -->
-        <visual>
+        <!-- <visual>
             <origin rpy="0 0 0" xyz="0 0 ${-link4_l/2}" />
             <geometry>
@@ -272,12 +272,12 @@
         <xacro:inertial_cylinder mass="${link4_mass}" length="${link4_l}" radius="${link4_r}">
             <origin rpy="0 0 0" xyz="0 0 ${-link4_l/2}" />
-        </xacro:inertial_cylinder>
-    </link>
-    <joint name="joint4" type="fixed">
+        </xacro:inertial_cylinder> -->
+    <!-- </link> -->
+    <!-- <joint name="joint4" type="fixed">
         <parent link="link3" />
         <child link="link4" />
         <origin rpy="${link4_alpha} 0 ${link4_theta}" xyz="0 0 ${link4_d}" />
         <axis xyz="0 0 1" />
-    </joint>
+    </joint> -->
     <!--
             Gazebo configuration
@@ -318,4 +318,9 @@
         </plugin>
         <plugin
+            filename="gz-sim-apply-joint-force-system"
+            name="gz::sim::systems::ApplyJointForce">
+            <joint_name>joint3</joint_name>
+        </plugin>
+        <plugin
             filename="gz-sim-pose-publisher-system"
             name="gz::sim::systems::PosePublisher">

Commit message: add assignement interface package

File: src/assign2/urdf/scara_fixed_joints.urdf.xacro (robot description, xacro)
@@ -253,5 +253,5 @@
         <axis xyz="0 0 -1" />
         <limit lower="${joint3_lower}" upper="${joint3_upper}" effort="1000" velocity="5" />
-        <dynamics damping="5" friction="100"/>
+        <dynamics damping="1" friction="0.5"/>
     </joint>
     <!-- <link name="link4"> -->

Commit message: changed friction to 0, damping to 1

File: src/assign2/urdf/scara_fixed_joints.urdf.xacro (robot description, xacro)
@@ -253,5 +253,5 @@
         <axis xyz="0 0 -1" />
         <limit lower="${joint3_lower}" upper="${joint3_upper}" effort="1000" velocity="5" />
-        <dynamics damping="1" friction="0.5"/>
+        <dynamics damping="1" friction="0"/>
     </joint>
     <!-- <link name="link4"> -->
