Commit message: Added velocity controller
Co-authored-by: Copilot <copilot@github.com>

File: src/assign3/urdf/scara_fixed_joints.urdf.xacro (robot description, xacro)
@@ -1,4 +1,5 @@
 <?xml version="1.0"?>
 <robot name="scara_robot" xmlns:xacro="http://www.ros.org/wiki/xacro">
+    <xacro:arg name="control_mode" default="velocity" />
     <!-- Joint colors-->
     <material name="blue">
@@ -40,10 +41,10 @@
     <xacro:property name="base_link_mass" value="100" />
     <!-- Joint 1 -->
-    <xacro:property name="joint1_lower" value="${-pi}" />
-    <xacro:property name="joint1_upper" value="${pi}" />
+    <xacro:property name="joint1_lower" value="${-7*pi/8}" />
+    <xacro:property name="joint1_upper" value="${7*pi/8}" />
     <!-- Joint 1 visual-->
     <xacro:property name="link1_l" value="${d1}" />
     <xacro:property name="link1_r" value="${cyl_joint_r}" />
-    <xacro:property name="link1_mass" value="1" />
+    <xacro:property name="link1_mass" value="10" />
     <!-- DH data of joint 1-->
     <xacro:property name="link1_theta" value="0" />
@@ -57,10 +58,10 @@
     <xacro:property name="link1_arm_mass" value="5" />
     <!-- Joint 1 -->
-    <xacro:property name="joint2_lower" value="${-pi}" />
-    <xacro:property name="joint2_upper" value="${pi}" />
+    <xacro:property name="joint2_lower" value="${-2*pi/3}" />
+    <xacro:property name="joint2_upper" value="${2*pi/3}" />
     <!-- Joint 2 visual-->
     <xacro:property name="link2_l" value="${cyl_joint_l}" />
     <xacro:property name="link2_r" value="${cyl_joint_r}" />
-    <xacro:property name="link2_mass" value="1" />
+    <xacro:property name="link2_mass" value="5" />
     <!-- DH data of joint 2-->
     <xacro:property name="link2_theta" value="0" />
@@ -72,5 +73,5 @@
     <xacro:property name="link2_arm_w" value="${link_arm_a}" />
     <xacro:property name="link2_arm_h" value="${link_arm_a}" />
-    <xacro:property name="link2_arm_mass" value="4" />
+    <xacro:property name="link2_arm_mass" value="5" />
     <!-- Joint 3 -->
     <!-- Prismatic extend limit -->
@@ -227,4 +228,5 @@
         <limit lower="${joint2_lower}" upper="${joint2_upper}" effort="100" velocity="1.0" />
         <axis xyz="0 0 1" />
+        <dynamics damping="1" friction="0"/>
     </joint>
     <link name="link3">
@@ -312,4 +314,6 @@
     </gazebo> -->
     <gazebo>
+    </gazebo>
+    <gazebo>
         <plugin
             filename="gz-sim-joint-state-publisher-system"
@@ -317,9 +321,43 @@
             <topic>/joint_states</topic>
         </plugin>
-        <plugin
-            filename="gz-sim-apply-joint-force-system"
-            name="gz::sim::systems::ApplyJointForce">
-            <joint_name>joint3</joint_name>
+        <!-- Force controllers -->
+        <xacro:if value="${'$(arg control_mode)' == 'force'}">
+            <plugin
+                filename="gz-sim-apply-joint-force-system"
+                name="gz::sim::systems::ApplyJointForce">
+                <joint_name>joint1</joint_name>
+            </plugin>
+            <plugin
+                filename="gz-sim-apply-joint-force-system"
+                name="gz::sim::systems::ApplyJointForce">
+                <joint_name>joint2</joint_name>
+            </plugin>
+            <plugin
+                filename="gz-sim-apply-joint-force-system"
+                name="gz::sim::systems::ApplyJointForce">
+                <joint_name>joint3</joint_name>
         </plugin>
+        </xacro:if>
+        <!-- Velocity controllers -->
+        <xacro:if value="${'$(arg control_mode)' == 'velocity'}">
+            <plugin
+                filename="gz-sim-joint-controller-system"
+                name="gz::sim::systems::JointController">
+                <joint_name>joint1</joint_name>
+                <initial_velocity>0.0</initial_velocity>
+            </plugin>
+            <plugin
+                filename="gz-sim-joint-controller-system"
+                name="gz::sim::systems::JointController">
+                <joint_name>joint2</joint_name>
+                <initial_velocity>0.0</initial_velocity>
+            </plugin>
+            <plugin
+                filename="gz-sim-joint-controller-system"
+                name="gz::sim::systems::JointController">
+                <joint_name>joint3</joint_name>
+                <initial_velocity>0.0</initial_velocity>
+            </plugin>
+        </xacro:if>
         <plugin
             filename="gz-sim-pose-publisher-system"

Commit message: Added velocity controller
Co-authored-by: Copilot <copilot@github.com>

File: src/assign3/urdf/scara_fixed_joints.urdf.xacro (robot description, xacro)
@@ -41,6 +41,6 @@
     <xacro:property name="base_link_mass" value="100" />
     <!-- Joint 1 -->
-    <xacro:property name="joint1_lower" value="${-7*pi/8}" />
-    <xacro:property name="joint1_upper" value="${7*pi/8}" />
+    <xacro:property name="joint1_lower" value="${-pi}" />
+    <xacro:property name="joint1_upper" value="${pi}" />
     <!-- Joint 1 visual-->
     <xacro:property name="link1_l" value="${d1}" />
@@ -150,5 +150,5 @@
         <axis xyz="0 0 1" />
         <limit lower="${joint1_lower}" upper="${joint1_upper}" effort="100" velocity="5.0" />
-        <dynamics damping="0.1" friction="0.0"/>
+        <dynamics damping="0.1" friction="100.0"/>
     </joint>
     <link name="link1">
@@ -228,5 +228,5 @@
         <limit lower="${joint2_lower}" upper="${joint2_upper}" effort="100" velocity="1.0" />
         <axis xyz="0 0 1" />
-        <dynamics damping="1" friction="0"/>
+        <dynamics damping="1" friction="100"/>
     </joint>
     <link name="link3">
