Commit message: revert the joint

File: src/assign3/urdf/scara_fixed_joints.urdf.xacro (robot description, xacro)
@@ -150,5 +150,5 @@
         <axis xyz="0 0 1" />
         <limit lower="${joint1_lower}" upper="${joint1_upper}" effort="100" velocity="5.0" />
-        <dynamics damping="0.1" friction="100.0"/>
+        <dynamics damping="0.1" friction="0"/>
     </joint>
     <link name="link1">
@@ -228,5 +228,5 @@
         <limit lower="${joint2_lower}" upper="${joint2_upper}" effort="100" velocity="1.0" />
         <axis xyz="0 0 1" />
-        <dynamics damping="1" friction="100"/>
+        <dynamics damping="1" friction="0"/>
     </joint>
     <link name="link3">
